File: hardware/Carte_puissance.kicad_sch (KiCad schematic)
At the start: 4 parts

Commit message: Erreur de manipulation, version 2.3 ok
Connections:
- no-connect marks 2 -> 0
Other:
- sheet IO ports: added none; removed ENCODER_A_PHB, ENCODER_B_PHB
Changed lines of the file:
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@@
 	(title_block
 		(title "ALAMAK Carte Puissance")
-		(date "2026-05-21")
-		(rev "2.0")
+		(date "2026-06-29")
+		(rev "2.3")
 		(company "INSA")
-	)
-	(no_connect
-		(at 139.7 153.67)
-	)
-	(no_connect
-		(at 139.7 156.21)
 	)
 	(wire
@@
 			)
 		)
-		(pin "ENCODER_B_PHB" output
-			(at 139.7 156.21 180)
-			(effects
-				(font
-					(size 1.27 1.27)
-				)
-				(justify left)
-			)
-		)
 		(pin "ENCODER_B_PHA" output
 			(at 139.7 124.46 180)
 			(effects
 				(font
-					(size 1.27 1.27)
-				)
-				(justify left)
-			)
-		)
-		(pin "ENCODER_A_PHB" output
-			(at 139.7 153.67 180)
-			(effects
-				(font
