File: hardware/cpu.kicad_sch (KiCad schematic)
At the start: 15 parts, among them J11 FTSH-105-01-L-DV-007-K-TR, U3 MCXA153VLH

Commit message: Erreur de manipulation, version 2.3 ok
Parts:
- added R16: 10K, Resistor_SMD:R_0805_2012Metric, symbol Device:R
- added SW1, SW2: SW_Push, Button_Switch_SMD:SW_SPST_EVQP2, symbol Switch:SW_Push
- R10, R7, R8: Part Number RT0805DRE07100RL -> RT0805FRE10100KL
Connections:
- net +3.3V: now also SW1.2
- net GND: now also R16.1, SW2.1
- net nRESET: now also SW2.2
- net at U3.30 (P3_31/LPTMR0_ALT2/TRIG_IN10/CT0_MAT3/ADC0_A12): now also R16.2, SW1.1
- no-connect marks 36 -> 35

Commit message: V2.3b: correction sur la nomenclature (bom) de plusieurs composants, suppression d'une mauvaise manipulation precedente
Parts:
- C17: Part Number CL21B105KBFNNNG -> CL21B105KBFNNNF
- C19: Part Number CL21B474KBFNNNE -> CL21B474KBFNNNG
- R16: Manufacturer Yageo -> Vishay; Part Number RT0805FRE10100KL -> RCA080510K0JNEASR
- R9: Part Number RT0805DRE07100RL -> RT0805FRE132K2L
- SW1, SW2: value SW_Push -> EVQ-P2602M; Manufacturer (none) -> Panasonic; Part Number (none) -> EVQ-P2602M
Changed lines of the file:
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@@
 	(title_block
 		(title "ALAMAK - CPU")
-		(date "2026-05-28")
-		(rev "2.1")
+		(date "2026-09-22")
+		(rev "2.3b")
 		(company "INSA - GEI")
 	)
@@
 			)
 		)
-		(property "Part Number" "CL21B474KBFNNNE"
+		(property "Part Number" "CL21B474KBFNNNG"
 			(at 200.66 99.06 0)
 			(effects
@@
 			)
 		)
-		(property "Value" "SW_Push"
+		(property "Value" "EVQ-P2602M"
 			(at 27.94 167.6399 90)
 			(effects
@@
 			)
 		)
+		(property "Manufacturer" "Panasonic"
+			(at 26.67 166.37 0)
+			(effects
+				(font
+					(size 1.27 1.27)
+				)
+				(hide yes)
+			)
+		)
+		(property "Part Number" "EVQ-P2602M"
+			(at 26.67 166.37 0)
+			(effects
+				(font
+					(size 1.27 1.27)
+				)
+				(hide yes)
+			)
+		)
 		(pin "1"
 		)
@@
 			)
 		)
-		(property "Part Number" "CL21B105KBFNNNG"
+		(property "Part Number" "CL21B105KBFNNNF"
 			(at 187.96 30.48 0)
 			(effects
@@
 			)
 		)
-		(property "Manufacturer" "Yageo"
+		(property "Manufacturer" "Vishay"
 			(at 21.59 175.26 0)
 			(effects
@@
 			)
 		)
-		(property "Part Number" "RT0805FRE10100KL"
+		(property "Part Number" "RCA080510K0JNEASR"
 			(at 21.59 175.26 0)
 			(effects
@@
 			)
 		)
-		(property "Value" "SW_Push"
+		(property "Value" "EVQ-P2602M"
 			(at 35.56 24.1299 90)
 			(effects
@@
 			)
 		)
+		(property "Manufacturer" "Panasonic"
+			(at 34.29 22.86 0)
+			(effects
+				(font
+					(size 1.27 1.27)
+				)
+				(hide yes)
+			)
+		)
+		(property "Part Number" "EVQ-P2602M"
+			(at 34.29 22.86 0)
+			(effects
+				(font
+					(size 1.27 1.27)
+				)
+				(hide yes)
+			)
+		)
 		(pin "1"
 		)
@@
 			)
 		)
-		(property "Part Number" "RT0805DRE07100RL"
+		(property "Part Number" "RT0805FRE132K2L"
 			(at 212.09 106.68 0)
 			(effects
