File: hardware/io.kicad_sch (KiCad schematic)
At the start: 34 parts, among them J10 Cable Servomoteur JST, J5 SeedStudio 110990037, J6 72454-010VLF, J7 DF3A-5P-2DS, J8 DF3A-5P-2DS, J9 B2B-XH-2, Q2 TPH2R506PL,L1Q, U4 PCA9306DP, U5 74AHC1G126

Commit message: Erreur de manipulation, version 2.3 ok
Parts:
- added JP5, JP6: Jumper_3_Open, Jumper:SolderJumper-3_P1.3mm_Open_RoundedPad1.0x1.5mm, symbol Jumper:Jumper_3_Open
- added R25, R26: 15K, Resistor_SMD:R_0805_2012Metric, symbol Device:R
- Q2: footprint Package_SO:SOP-8_5.28x5.23mm_P1.27mm -> Package_SO:SOP-8_3.76x4.96mm_P1.27mm
- R11, R21: Part Number RT0805DRE07100RL -> RT0805FRE10100KL
- R22, R23: value 100R -> 10K; Part Number RT0805DRE07100RL -> RT0805FRE10100KL
Connections:
- net +3.3V: now also JP5.1 (A), JP6.1 (A); no longer J7.2, J8.2
- net +5V: now also JP5.3 (B), JP6.3 (B)
- net ENCODER_A_PHA: now also R25.2
- net ENCODER_B_PHA: now also R26.2
- net GND: now also R25.1, R26.1
- net ENCODER_A_PHB: no longer names the net of J7.4
- net ENCODER_B_PHB: no longer names the net of J8.4
- new net: J8.2, JP6.2 (C)
- new net: J7.2, JP5.2 (C)
- no-connect marks 7 -> 9
Other:
- note added: "ATTENTION Penser à relier le 5V ou 3V3"
- moved on the sheet: R22, R23

Commit message: V2.3b: correction sur la nomenclature (bom) de plusieurs composants, suppression d'une mauvaise manipulation precedente
Parts:
- C25, C26: Part Number CL21B105KBFNNNG -> CL21B105KBFNNNF
- C27: Manufacturer Murata -> TDK; Part Number GRM21BR61H106KE43L -> CGA4J1X7S1E106K125AE
- JP5, JP6: Manufacturer (none) -> -; Part Number (none) -> -
- R11, R21: Part Number RT0805FRE10100KL -> RT0805DRE07100RL
- R22, R23: Manufacturer Yageo -> Vishay; Part Number RT0805FRE10100KL -> RCA080510K0JNEASR
- R25, R26: Part Number RT0805FRE10100KL -> RT0805DRE0715KL
- TP1, TP15: value Conn_01x03_Pin -> TestPoint
- U4: Part Number PCA9306DP -> PCA9306DP,118
Changed lines of the file:
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@@
 	(title_block
 		(title "ALAMAK - IO")
-		(date "2026-05-21")
-		(rev "2.0")
+		(date "2026-09-22")
+		(rev "2.3b")
 		(company "INSA - GEI")
 	)
@@
 			)
 		)
-		(property "Manufacturer" "Yageo"
+		(property "Manufacturer" "Vishay"
 			(at 210.82 39.37 0)
 			(effects
@@
 			)
 		)
-		(property "Part Number" "RT0805FRE10100KL"
+		(property "Part Number" "RCA080510K0JNEASR"
 			(at 210.82 39.37 0)
 			(effects
@@
 			)
 		)
-		(property "Part Number" "PCA9306DP"
+		(property "Part Number" "PCA9306DP,118"
 			(at 41.91 74.93 0)
 			(effects
@@
 			)
 		)
+		(property "Manufacturer" "-"
+			(at 219.71 21.59 0)
+			(effects
+				(font
+					(size 1.27 1.27)
+				)
+				(hide yes)
+			)
+		)
+		(property "Part Number" "-"
+			(at 219.71 21.59 0)
+			(effects
+				(font
+					(size 1.27 1.27)
+				)
+				(hide yes)
+			)
+		)
 		(pin "1"
 		)
@@
 			)
 		)
-		(property "Manufacturer" "Murata"
+		(property "Manufacturer" "TDK"
 			(at 82.55 175.26 0)
 			(effects
@@
 			)
 		)
-		(property "Part Number" "GRM21BR61H106KE43L"
+		(property "Part Number" "CGA4J1X7S1E106K125AE"
 			(at 82.55 175.26 0)
 			(effects
@@
 			)
 		)
-		(property "Manufacturer" "Yageo"
+		(property "Manufacturer" "Vishay"
 			(at 210.82 88.9 0)
 			(effects
@@
 			)
 		)
-		(property "Part Number" "RT0805FRE10100KL"
+		(property "Part Number" "RCA080510K0JNEASR"
 			(at 210.82 88.9 0)
 			(effects
@@
 			)
 		)
-		(property "Value" "Conn_01x03_Pin"
+		(property "Value" "TestPoint"
 			(at 131.445 181.61 0)
 			(effects
@@
 			)
 		)
-		(property "Part Number" "RT0805FRE10100KL"
+		(property "Part Number" "RT0805DRE07100RL "
 			(at 83.82 69.85 0)
 			(effects
@@
 			)
 		)
-		(property "Part Number" "CL21B105KBFNNNG"
+		(property "Part Number" "CL21B105KBFNNNF"
 			(at 107.95 124.46 0)
 			(effects
@@
 			)
 		)
-		(property "Part Number" "RT0805FRE10100KL"
+		(property "Part Number" "RT0805DRE07100RL "
 			(at 82.55 168.91 0)
 			(effects
@@
 			)
 		)
-		(property "Part Number" "CL21B105KBFNNNG"
+		(property "Part Number" "CL21B105KBFNNNF"
 			(at 29.21 38.1 0)
 			(effects
@@
 			)
 		)
-		(property "Value" "Conn_01x03_Pin"
+		(property "Value" "TestPoint"
 			(at 131.445 161.29 0)
 			(effects
@@
 			)
 		)
-		(property "Part Number" "RT0805FRE10100KL"
+		(property "Part Number" "RT0805DRE0715KL"
 			(at 215.9 43.18 0)
 			(effects
@@
 			)
 		)
+		(property "Manufacturer" "-"
+			(at 220.98 71.12 0)
+			(effects
+				(font
+					(size 1.27 1.27)
+				)
+				(hide yes)
+			)
+		)
+		(property "Part Number" "-"
+			(at 220.98 71.12 0)
+			(effects
+				(font
+					(size 1.27 1.27)
+				)
+				(hide yes)
+			)
+		)
 		(pin "1"
 		)
@@
 			)
 		)
-		(property "Part Number" "RT0805FRE10100KL"
+		(property "Part Number" "RT0805DRE0715KL"
 			(at 217.17 92.71 0)
 			(effects
