File: hardware/puissance.kicad_sch (KiCad schematic)
At the start: 49 parts, among them J1 Cable XT60, J2 B2B-XH-2, J3 B2PS-VH, J4 B2PS-VH, Q1 IPD50P04P413ATMA2, Q3 IPD30N03S4L-09, Q4 IPD30N03S4L-09, U1 LTC2954CTS8-2#TRMPBF, U2 MIC4427

Commit message: Erreur de manipulation, version 2.3 ok
Parts:
- added JP4: SolderJumper_2_Open, Jumper:SolderJumper-2_P1.3mm_Open_RoundedPad1.0x1.5mm, symbol Jumper:SolderJumper_2_Open
- R2: value 100K -> 10R
Connections:
- net ~{ONOFF_KILL}: now also JP4.2 (B); no longer U1.8 (~{KILL})
- new net: JP4.1 (A), U1.8 (~{KILL})
Changed lines of the file:
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@@
 	(wire
 		(pts
+			(xy 121.92 53.34) (xy 121.92 48.26)
+		)
+		(stroke
+			(width 0)
+			(type default)
+		)
+	)
+	(wire
+		(pts
 			(xy 66.04 172.72) (xy 66.04 175.26)
 		)
@@
 	(wire
 		(pts
-			(xy 111.76 48.26) (xy 115.57 48.26)
+			(xy 121.92 53.34) (xy 129.54 53.34)
 		)
 		(stroke
@@
 	(wire
 		(pts
+			(xy 111.76 48.26) (xy 114.3 48.26)
+		)
+		(stroke
+			(width 0)
+			(type default)
+		)
+	)
+	(wire
+		(pts
 			(xy 80.01 29.21) (xy 81.28 29.21)
 		)
@@
 	(hierarchical_label "~{ONOFF_KILL}"
 		(shape input)
-		(at 115.57 48.26 0)
+		(at 129.54 53.34 0)
 		(effects
 			(font
@@
 	)
 	(symbol
+		(lib_id "Jumper:SolderJumper_2_Open")
+		(at 118.11 48.26 0)
+		(unit 1)
+		(exclude_from_sim yes)
+		(in_bom no)
+		(on_board yes)
+		(dnp no)
+		(property "Reference" "JP4"
+			(at 118.11 46.228 0)
+			(effects
+				(font
+					(size 1.27 1.27)
+				)
+			)
+		)
+		(property "Value" "SolderJumper_2_Open"
+			(at 118.11 44.45 0)
+			(effects
+				(font
+					(size 1.27 1.27)
+				)
+				(hide yes)
+			)
+		)
+		(property "Footprint" "Jumper:SolderJumper-2_P1.3mm_Open_RoundedPad1.0x1.5mm"
+			(at 118.11 48.26 0)
+			(effects
+				(font
+					(size 1.27 1.27)
+				)
+				(hide yes)
+			)
+		)
+		(property "Datasheet" "~"
+			(at 118.11 48.26 0)
+			(effects
+				(font
+					(size 1.27 1.27)
+				)
+				(hide yes)
+			)
+		)
+		(property "Description" "Solder Jumper, 2-pole, open"
+			(at 118.11 48.26 0)
+			(effects
+				(font
+					(size 1.27 1.27)
+				)
+				(hide yes)
+			)
+		)
+		(pin "1"
+		)
+		(pin "2"
+		)
+		(instances
+			(project ""
+				(path "/aaa0f7a4-a021-413b-80cf-aab59bb3339a/79ff172e-6092-41ef-91e3-a41ed4e55444"
+					(reference "JP4")
+					(unit 1)
+				)
+			)
+		)
+	)
+	(symbol
 		(lib_id "power:GNDPWR")
 		(at 123.19 133.35 0)
@@
 			)
 		)
-		(property "Value" "100K"
+		(property "Value" "10R"
 			(at 138.303 44.958 0)
 			(effects

Commit message: V2.3b: correction sur la nomenclature (bom) de plusieurs composants, suppression d'une mauvaise manipulation precedente
Parts:
- C1: Part Number CL21B105KBFNNNG -> CL21B105KBFNNNF
- C11, C3, C6, C9: Manufacturer Murata -> TDK; Part Number GRM21BR61H106KE43L -> CGA4J1X7S1E106K125AE
- JP4: Manufacturer (none) -> -; Part Number (none) -> -
- R2: Part Number RT0805FRE10100KL -> RT0805FRE1310RL
- U1: Part Number LTC2954CTS8-2#TRMPBF -> LTC2954CTS8-2#TRPBF
- U2: Part Number MIC4427 -> MIC4427ZM
Other:
- company: (none) -> INSA-GEI
- title: (none) -> Puissance
Changed lines of the file:
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@@
 	(generator_version "8.0")
 	(paper "A4")
+	(title_block
+		(title "Puissance")
+		(date "2026-09-22")
+		(rev "2.3b")
+		(company "INSA-GEI")
+	)
 	(junction
 		(at 129.54 29.21)
@@
 			)
 		)
-		(property "Part Number" "CL21B105KBFNNNG"
+		(property "Part Number" "CL21B105KBFNNNF"
 			(at 113.03 55.88 0)
 			(effects
@@
 			)
 		)
-		(property "Part Number" "LTC2954CTS8-2#TRMPBF"
+		(property "Part Number" "LTC2954CTS8-2#TRPBF"
 			(at 81.28 40.64 0)
 			(effects
@@
 			)
 		)
-		(property "Manufacturer" "Murata"
+		(property "Manufacturer" "TDK"
 			(at 53.34 179.07 0)
 			(effects
@@
 			)
 		)
-		(property "Part Number" "GRM21BR61H106KE43L"
+		(property "Part Number" "CGA4J1X7S1E106K125AE"
 			(at 53.34 179.07 0)
 			(effects
@@
 			)
 		)
+		(property "Manufacturer" "-"
+			(at 118.11 48.26 0)
+			(effects
+				(font
+					(size 1.27 1.27)
+				)
+				(hide yes)
+			)
+		)
+		(property "Part Number" "-"
+			(at 118.11 48.26 0)
+			(effects
+				(font
+					(size 1.27 1.27)
+				)
+				(hide yes)
+			)
+		)
 		(pin "1"
 		)
@@
 			)
 		)
-		(property "Part Number" "MIC4427"
+		(property "Part Number" "MIC4427ZM"
 			(at 123.19 115.57 0)
 			(effects
@@
 			)
 		)
-		(property "Part Number" "RT0805FRE10100KL"
+		(property "Part Number" "RT0805FRE1310RL"
 			(at 137.16 43.18 0)
 			(effects
@@
 			)
 		)
-		(property "Manufacturer" "Murata"
+		(property "Manufacturer" "TDK"
 			(at 63.5 125.73 0)
 			(effects
@@
 			)
 		)
-		(property "Part Number" "GRM21BR61H106KE43L"
+		(property "Part Number" "CGA4J1X7S1E106K125AE"
 			(at 63.5 125.73 0)
 			(effects
@@
 			)
 		)
-		(property "Manufacturer" "Murata"
+		(property "Manufacturer" "TDK"
 			(at 187.96 39.37 0)
 			(effects
@@
 			)
 		)
-		(property "Part Number" "GRM21BR61H106KE43L"
+		(property "Part Number" "CGA4J1X7S1E106K125AE"
 			(at 187.96 39.37 0)
 			(effects
@@
 			)
 		)
-		(property "Manufacturer" "Murata"
+		(property "Manufacturer" "TDK"
 			(at 129.54 152.4 0)
 			(effects
@@
 			)
 		)
-		(property "Part Number" "GRM21BR61H106KE43L"
+		(property "Part Number" "CGA4J1X7S1E106K125AE"
 			(at 129.54 152.4 0)
 			(effects
