File: hardware/Carte_puissance.kicad_pcb (KiCad board)
At the start: 4 copper layers, 124 x 62 mm, 102 parts, among them J1 Cable XT60, J10 Cable Servomoteur JST, J11 FTSH-105-01-L-DV-007-K-TR, J2 B2B-XH-2, J3 B2PS-VH, J4 B2PS-VH, J5 SeedStudio 110990037, J6 72454-010VLF, J7 DF3A-5P-2DS, J8 DF3A-5P-2DS, J9 B2B-XH-2, Q1 IPD50P04P413ATMA2, Q2 TPH2R506PL,L1Q, Q3 IPD30N03S4L-09, Q4 IPD30N03S4L-09, U1 LTC2954CTS8-2#TRMPBF, U2 MIC4427, U3 MCXA153VLH, U4 PCA9306DP, U5 74AHC1G126

Commit message: Erreur de manipulation, version 2.3 ok
Parts:
- added JP4: SolderJumper_2_Open, Jumper:SolderJumper-2_P1.3mm_Open_RoundedPad1.0x1.5mm, B.Cu at (160.6, 122.1)
- added JP5: Jumper_3_Open, Jumper:SolderJumper-3_P1.3mm_Open_RoundedPad1.0x1.5mm, B.Cu at (200.2, 143.4)
- added JP6: Jumper_3_Open, Jumper:SolderJumper-3_P1.3mm_Open_RoundedPad1.0x1.5mm, B.Cu at (128.6, 143.4)
- added R16: 10K, Resistor_SMD:R_0805_2012Metric, F.Cu at (195.5, 127.7)
- added R25: 15K, Resistor_SMD:R_0805_2012Metric, F.Cu at (187.1, 139.9)
- added R26: 15K, Resistor_SMD:R_0805_2012Metric, F.Cu at (126.5, 139.9)
- added SW1: SW_Push, Button_Switch_SMD:SW_SPST_EVQP2, F.Cu at (195.6, 132.8)
- added SW2: SW_Push, Button_Switch_SMD:SW_SPST_EVQP2, F.Cu at (132.6, 132.8)
- Q2: footprint Package_SO:SOP-8_5.28x5.23mm_P1.27mm -> Package_SO:SOP-8_3.76x4.96mm_P1.27mm
- R14, R15: moved to F.Cu
- R2: value 100K -> 10R
- R22, R23: value 100R -> 10K
- moved TP1 46.1 mm to (179.5, 132.1)
- moved R10 15.8 mm to (194.1, 107.4), turned to 90 degrees
- moved C16 14.5 mm to (199.0, 99.1), turned to 90 degrees
- moved C19 11.5 mm to (184.4, 113.9)
- moved R7 10.7 mm to (185.1, 110.4), turned to 180 degrees
- moved J11 7.81 mm to (191.8, 114.0)
- moved R8 7.81 mm to (199.3, 109.5)
- moved R9 7.81 mm to (199.3, 112.5)
- moved U4 5.27 mm to (119.4, 124.2), turned to 180 degrees
- moved R14 4.33 mm to (103.7, 112.9)
- moved R15 4.33 mm to (103.7, 109.9)
- moved J9 3.61 mm to (210.6, 97.2)
- moved Q2 3.61 mm to (211.9, 104.8)
- moved C25 2.89 mm to (102.2, 100.8)
- moved R12 2.89 mm to (109.3, 100.8)
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Connections:
- J7 pad 2: +3.3V -> Net-(JP5-C)
- J7 pad 4: /IO/ENCODER_A_PHB -> unconnected-(J7-Pad4)
- J8 pad 2: +3.3V -> Net-(JP6-C)
- J8 pad 4: /IO/ENCODER_B_PHB -> unconnected-(J8-Pad4)
- U1 pad 8: /CPU/~{ONOFF_KILL} -> Net-(JP4-A)
- U3 pad 30: unconnected-(U3-P3_31/LPTMR0_ALT2/TRIG_IN10/CT0_MAT3/ADC0_A12-Pad30) -> Net-(U3-P3_31/LPTMR0_ALT2/TRIG_IN10/CT0_MAT3/ADC0_A12)
Routing:
- net +5V: track 53.6 -> 223.9 mm, vias 0 -> 1
- net Net-(U3-P3_31/LPTMR0_ALT2/TRIG_IN10/CT0_MAT3/ADC0_A12): track 0.00 -> 57.3 mm
- net /CPU/I2C_SCL: track 74.0 -> 113.6 mm, vias 0 -> 1
- net /CPU/I2C_SDA: track 85.6 -> 115.2 mm, vias 0 -> 1
- net /CPU/nRESET: track 64.5 -> 92.2 mm, vias 2 -> 0
- net GNDPWR: track 408.8 -> 384.2 mm, vias 76 -> 86
- net Net-(U2-OUT_A): track 46.9 -> 63.6 mm
- net GND: track 109.2 -> 123.7 mm, vias 22 -> 25
- net /CPU/SWCLK: track 46.4 -> 59.0 mm, vias 2 -> 3
- net +3.3V: track 73.0 -> 84.5 mm, vias 11 -> 13
- net Net-(JP5-C): track 0.00 -> 8.72 mm
- net /CPU/SWO: track 41.3 -> 49.5 mm, vias 0 -> 2
- net +BATT: track 202.5 -> 194.5 mm
- net Net-(JP4-A): track 0.00 -> 7.95 mm, vias 0 -> 1
- net Net-(JP6-C): track 0.00 -> 7.83 mm
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Other:
- board text added: "3V"
- board text added: "TP1: I2C TP2: PWM-SERVO TP3: PHA-ENC A TP4: PHA-ENC B TP5: MESURE-VBAT TP6: PWM-MOT A TP7: PWM-MOT B"
- board text added: "TP9: 5V TP10: ENABLE Q1 TP11: ~{ONOFF_INT} TP12: ~{ONOFF_KILL} TP13: GND TP14: GNDPWR TP15: DEBUG-UART"
- board text removed: "TP1: I2C TP2: PWM-SERVO TP3: PHA-ENC A TP4: PHA-ENC B TP5: MESURE-VBAT TP6: PWM-MOT A TP7: PWM-MOT B TP8: 3V3 TP9: 5V TP10: ENABLE Q1 TP11: ~{ONOFF_INT} TP12: ~{ONOFF_KILL} TP13: GND TP14: GNDPWR TP15: DEBUG-UART"

Commit message: Corrections sur la carte puissance
Parts:
- SW1, SW2: value SW_Push -> EVQ-P2602M
- TP1, TP15: value Conn_01x03_Pin -> TestPoint
Changed lines of the file:
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@@
 			)
 		)
-		(property "Part Number" "CL21B474KBFNNNE"
+		(property "Part Number" "CL21B474KBFNNNG"
 			(at 0 0 -90)
 			(unlocked yes)
@@
 			)
 		)
-		(property "Value" "SW_Push"
+		(property "Value" "EVQ-P2602M"
 			(at 0 3 90)
 			(layer "F.Fab")
@@
 			)
 		)
+		(property "Manufacturer" "Panasonic"
+			(at 0 0 90)
+			(unlocked yes)
+			(layer "F.Fab")
+			(hide yes)
+			(effects
+				(font
+					(size 1 1)
+					(thickness 0.15)
+				)
+			)
+		)
+		(property "Part Number" "EVQ-P2602M"
+			(at 0 0 90)
+			(unlocked yes)
+			(layer "F.Fab")
+			(hide yes)
+			(effects
+				(font
+					(size 1 1)
+					(thickness 0.15)
+				)
+			)
+		)
 		(sheetname "CPU")
 		(sheetfile "cpu.kicad_sch")
@@
 			)
 		)
-		(property "Manufacturer" "Murata"
+		(property "Manufacturer" "TDK"
 			(at 0 0 0)
 			(unlocked yes)
@@
 			)
 		)
-		(property "Part Number" "GRM21BR61H106KE43L"
+		(property "Part Number" "CGA4J1X7S1E106K125AE"
 			(at 0 0 0)
 			(unlocked yes)
@@
 			)
 		)
-		(property "Manufacturer" "Yageo"
+		(property "Manufacturer" "Vishay"
 			(at 0 0 180)
 			(unlocked yes)
@@
 			)
 		)
-		(property "Part Number" "RT0805FRE10100KL"
+		(property "Part Number" "RCA080510K0JNEASR"
 			(at 0 0 180)
 			(unlocked yes)
@@
 			)
 		)
-		(property "Value" "SW_Push"
+		(property "Value" "EVQ-P2602M"
 			(at 0 3 90)
 			(layer "F.Fab")
@@
 			)
 		)
+		(property "Manufacturer" "Panasonic"
+			(at 0 0 90)
+			(unlocked yes)
+			(layer "F.Fab")
+			(hide yes)
+			(effects
+				(font
+					(size 1 1)
+					(thickness 0.15)
+				)
+			)
+		)
+		(property "Part Number" "EVQ-P2602M"
+			(at 0 0 90)
+			(unlocked yes)
+			(layer "F.Fab")
+			(hide yes)
+			(effects
+				(font
+					(size 1 1)
+					(thickness 0.15)
+				)
+			)
+		)
 		(sheetname "CPU")
 		(sheetfile "cpu.kicad_sch")
@@
 			)
 		)
-		(property "Part Number" "RT0805FRE10100KL"
+		(property "Part Number" "RT0805DRE07100RL "
 			(at 0 0 0)
 			(unlocked yes)
@@
 			)
 		)
-		(property "Value" "Conn_01x03_Pin"
+		(property "Value" "TestPoint"
 			(at 0 7.41 0)
 			(layer "F.Fab")
@@
 			)
 		)
-		(property "Part Number" "PCA9306DP"
+		(property "Part Number" "PCA9306DP,118"
 			(at 0 0 180)
 			(unlocked yes)
@@
 			)
 		)
-		(property "Part Number" "CL21B105KBFNNNG"
+		(property "Part Number" "CL21B105KBFNNNF"
 			(at 0 0 0)
 			(unlocked yes)
@@
 			)
 		)
-		(property "Manufacturer" "Yageo"
+		(property "Manufacturer" "Vishay"
 			(at 0 0 0)
 			(unlocked yes)
@@
 			)
 		)
-		(property "Part Number" "RT0805FRE10100KL"
+		(property "Part Number" "RCA080510K0JNEASR"
 			(at 0 0 0)
 			(unlocked yes)
@@
 			)
 		)
-		(property "Value" "Conn_01x03_Pin"
+		(property "Value" "TestPoint"
 			(at 0 7.41 0)
 			(layer "F.Fab")
@@
 			)
 		)
-		(property "Part Number" "RT0805DRE07100RL"
+		(property "Part Number" "RT0805FRE132K2L"
 			(at 0 0 180)
 			(unlocked yes)
@@
 			)
 		)
-		(property "Manufacturer" "Yageo"
+		(property "Manufacturer" "Vishay"
 			(at 0 0 180)
 			(unlocked yes)
@@
 			)
 		)
-		(property "Part Number" "RT0805FRE10100KL"
+		(property "Part Number" "RCA080510K0JNEASR"
 			(at 0 0 180)
 			(unlocked yes)
@@
 			)
 		)
-		(property "Manufacturer" "Murata"
+		(property "Manufacturer" "TDK"
 			(at 0 0 90)
 			(unlocked yes)
@@
 			)
 		)
-		(property "Part Number" "GRM21BR61H106KE43L"
+		(property "Part Number" "CGA4J1X7S1E106K125AE"
 			(at 0 0 90)
 			(unlocked yes)
@@
 			)
 		)
-		(property "Manufacturer" "Murata"
+		(property "Manufacturer" "TDK"
 			(at 0 0 90)
 			(unlocked yes)
@@
 			)
 		)
-		(property "Part Number" "GRM21BR61H106KE43L"
+		(property "Part Number" "CGA4J1X7S1E106K125AE"
 			(at 0 0 90)
 			(unlocked yes)
@@
 			)
 		)
-		(property "Part Number" "RT0805FRE10100KL"
+		(property "Part Number" "RT0805DRE0715KL"
 			(at 0 0 180)
 			(unlocked yes)
@@
 			)
 		)
-		(property "Part Number" "RT0805FRE10100KL"
+		(property "Part Number" "RT0805FRE1310RL"
 			(at 0 0 0)
 			(unlocked yes)
@@
 			)
 		)
-		(property "Part Number" "CL21B105KBFNNNG"
+		(property "Part Number" "CL21B105KBFNNNF"
 			(at 0 0 180)
 			(unlocked yes)
@@
 			)
 		)
-		(property "Part Number" "CL21B105KBFNNNG"
+		(property "Part Number" "CL21B105KBFNNNF"
 			(at 0 0 -90)
 			(unlocked yes)
@@
 			)
 		)
-		(property "Manufacturer" "Murata"
+		(property "Manufacturer" "TDK"
 			(at 0 0 180)
 			(unlocked yes)
@@
 			)
 		)
-		(property "Part Number" "GRM21BR61H106KE43L"
+		(property "Part Number" "CGA4J1X7S1E106K125AE"
 			(at 0 0 180)
 			(unlocked yes)
@@
 			)
 		)
-		(property "Part Number" "MIC4427"
+		(property "Part Number" "MIC4427ZM"
 			(at 0 0 0)
 			(unlocked yes)
@@
 			)
 		)
-		(property "Part Number" "RT0805FRE10100KL"
+		(property "Part Number" "RT0805DRE07100RL "
 			(at 0 0 0)
 			(unlocked yes)
@@
 			)
 		)
-		(property "Part Number" "RT0805FRE10100KL"
+		(property "Part Number" "RT0805DRE0715KL"
 			(at 0 0 0)
 			(unlocked yes)
@@
 			)
 		)
-		(property "Part Number" "LTC2954CTS8-2#TRMPBF"
+		(property "Part Number" "LTC2954CTS8-2#TRPBF"
 			(at 0 0 0)
 			(unlocked yes)
@@
 			)
 		)
-		(property "Part Number" "CL21B105KBFNNNG"
+		(property "Part Number" "CL21B105KBFNNNF"
 			(at 0 0 90)
 			(unlocked yes)
@@
 			)
 		)
+		(property "Manufacturer" "-"
+			(at 0 0 -90)
+			(unlocked yes)
+			(layer "B.Fab")
+			(hide yes)
+			(effects
+				(font
+					(size 1 1)
+					(thickness 0.15)
+				)
+				(justify mirror)
+			)
+		)
+		(property "Part Number" "-"
+			(at 0 0 -90)
+			(unlocked yes)
+			(layer "B.Fab")
+			(hide yes)
+			(effects
+				(font
+					(size 1 1)
+					(thickness 0.15)
+				)
+				(justify mirror)
+			)
+		)
 		(property ki_fp_filters "Jumper* TestPoint*3Pads* TestPoint*Bridge*")
 		(sheetname "IO")
@@
 			)
 		)
+		(property "Manufacturer" "-"
+			(at 0 0 -90)
+			(unlocked yes)
+			(layer "B.Fab")
+			(hide yes)
+			(effects
+				(font
+					(size 1 1)
+					(thickness 0.15)
+				)
+				(justify mirror)
+			)
+		)
+		(property "Part Number" "-"
+			(at 0 0 -90)
+			(unlocked yes)
+			(layer "B.Fab")
+			(hide yes)
+			(effects
+				(font
+					(size 1 1)
+					(thickness 0.15)
+				)
+				(justify mirror)
+			)
+		)
 		(property ki_fp_filters "SolderJumper*Open*")
 		(sheetname "Puissance")
@@
 			)
 		)
-		(property "Manufacturer" "Murata"
+		(property "Manufacturer" "TDK"
 			(at 0 0 0)
 			(unlocked yes)
@@
 			)
 		)
-		(property "Part Number" "GRM21BR61H106KE43L"
+		(property "Part Number" "CGA4J1X7S1E106K125AE"
 			(at 0 0 0)
 			(unlocked yes)
@@
 					(thickness 0.15)
 				)
+				(justify mirror)
+			)
+		)
+		(property "Manufacturer" "-"
+			(at 0 0 -90)
+			(unlocked yes)
+			(layer "B.Fab")
+			(hide yes)
+			(effects
+				(font
+					(size 1 1)
+					(thickness 0.15)
+				)
+				(justify mirror)
+			)
+		)
+		(property "Part Number" "-"
+			(at 0 0 -90)
+			(unlocked yes)
+			(layer "B.Fab")
+			(hide yes)
+			(effects
+				(font
+					(size 1 1)
+					(thickness 0.15)
+				)
